Commit message: Fix URDF: set left wheel to symmetric position (0, 0.09, 0)

File: src/mks_motor_control/mks_motor_control/URDF/two_wheel_robot.urdf (robot description, URDF)
Before this commit: robot two_wheel_robot, 3 links, 2 joints
Joints:
- joint left_wheel_joint: origin xyz=0 0 0 rpy=0 0 0 -> xyz=0 0.09 0 rpy=0 0 0

Commit message: d

File: src/mks_motor_control/mks_motor_control/URDF/two_wheel_robot.urdf (robot description, URDF)
Before this commit: robot two_wheel_robot, 3 links, 2 joints
Links:
- link left_wheel_link: geometry visual cylinder length=0.01 radius=0.0425
- link right_wheel_link: geometry visual cylinder length=0.01 radius=0.0425

Commit message: Add LiDAR Unitree L2 with 112.5° pitch angle to URDF
- Add laser_frame link (LiDAR scanner geometry)
- Add lidar_joint with fixed type and 112.5° pitch angle
- Position: 10cm forward, 20cm up from base_link
- Pitch: 1.9635 radians (112.5 degrees) for table edge detection
- Enables precise LiDAR-based edge detection for hybrid localization
- Improves precision to ±6-8cm in RViz2 and Nav2 stack

Configuration Details:
- xyz: position relative to base_link (0.1m forward, 0m side, 0.2m up)
- rpy: roll=0°, pitch=112.5° (1.9635 rad), yaw=0°
- Type: fixed joint (no moving parts)

File: src/mks_motor_control/mks_motor_control/URDF/two_wheel_robot.urdf (robot description, URDF)
Before this commit: robot two_wheel_robot, 3 links, 2 joints
Links:
- added link laser_frame; visual cylinder length=0.05 radius=0.04
Joints:
- added joint lidar_joint: type fixed, parent base_link, child laser_frame, origin xyz=0.1 0.0 0.2 rpy=0 1.9635 0

Commit message: Update

File: src/mks_motor_control/mks_motor_control/URDF/two_wheel_robot.urdf (robot description, URDF)
Before this commit: robot two_wheel_robot, 4 links, 3 joints
Links:
- removed link laser_frame
Joints:
- removed joint lidar_joint
